File: cores/mzone/sch/megazone.kicad_sch (KiCad schematic)
At the start: 25 parts

Commit message: mzone core sch
Connections:
- net ~{MBS}: now reaches B_F14.18 (O0a)
- net MBS: now reaches B_F14.2 (I0a)

Commit message: mzone core
Other:
- added sheet IO (io.kicad_sch)

Commit message: mzone core
Other:
- sheet Slave CPU renamed Sub CPU
Changed lines of the file:
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@@
 			(color 0 0 0 0.0000)
 		)
-		(property "Sheetname" "Slave CPU"
+		(property "Sheetname" "Sub CPU"
 			(at 24.13 184.7084 0)
 			(effects

Commit message: mzone core
Parts:
- removed B_C13: 74LS08, symbol jt74:74LS08
- removed B_DE11: 74LS02, symbol jt74:74LS02
- removed B_DE13: 74LS00, symbol jt74:74LS00
Other:
- moved on the sheet: B_DE12B, C1B, C1C, C43, DE18A, E4A, F3B, G3A, G3B, G3D
