File: cores/mzone/sch/mcpu.kicad_sch (KiCad schematic)
At the start: 44 parts

Commit message: mzone core
Parts:
- removed unit 2 of B17
- removed unit 5 of B_A14
- removed B_B14, B_F14: 74LS240, symbol jt74:74LS240
- removed B_D10: 74LS244, symbol jt74:74LS244
- removed unit 1 of B_D14
- removed unit 7 of B_D14
- removed B_D8: 501, symbol skutis-kicad:501
- removed unit 2 of B_DE9
- removed B_F6, B_G6, B_G7: 74LS157, symbol jt74:74LS157
- removed B_F9: 74LS245, symbol jt74:74LS245
- removed B_G8: SRAM2K8B, symbol jt_ram:SRAM2K8B
- removed C17: 74LS240, symbol 74xx:74LS240_Split
- removed C40: 10n, symbol Device:C
- removed C43: 47n, symbol Device:C
- removed R47: 47R, symbol Device:R
- added B_B14, B_F14: 74LS240, symbol 74xx:74LS240_Split
- added B_D10: 74LS244, symbol 74xx:74LS244_Split
Connections:
- net H1'' is gone; now on net H1M: B_C10.11 (C), B_D14.6
- net H2''' is gone; now on net H2M: B_C10.12 (D), B_D14.4, B_DE9.12
- net INTST' is gone; now on an unnamed net: B_A13.12 (Q7)
- net AB0: now also B_F14.13
- net AB1: now also B_F14.11
- net AB2: now also B_F14.8
- net CLKE: now also B_D10.14
- net CLKQ: now also B_D10.16
- net COLRAM: now also B_B14.16
- net GND: now also B_B14.1, B_B14.19, B_F14.1, B_F14.15, B_F14.19, B_F14.6
- net INTSND: now also B_A14.16
- net INTST: now also B_A14.14
- net MBS: now also B_F14.2
- net MRD: now also B_B14.11, B_D10.12
- net MR~{W}: now also B_D10.8
- net MWR: now also B_B14.9
- net OBJRAM: now also B_B14.5
- net SCROLLX: now also B_B14.7
- net SCROLLY: now also B_B14.14
- net VRAM: now also B_B14.18
- net ~{AB}0: now also B_F14.7
- net ~{AB}1: now also B_F14.9
- net ~{AB}2: now also B_F14.12
- net ~{CLKQ}: now also B_D10.4
- net ~{COLRAM}: now also B_B14.4
- net ~{SCROLLX}: now also B_B14.13
- net ~{SCROLLY}: now also B_B14.6
- net ~{VRAM}: now also B_B14.2
- net at B_A13.7 (Q3): now also B_A14.4
- net at B_A14.13: now also B17.3
- net H2M: now reaches B_A14.7
- net H2M: now also B_D10.6
- net at B17.18: now also B_A14.15
- net H1M: now reaches B_A14.5
- net FLIP' renamed FLIP
- net ~{H2'''}: no longer names the net of B17.7, G17.19 (~{CE})
- net ~{H2''} renamed ~{H2}
- net ~{H2'}: no longer names the net of B_B12.13, B_B12.2, B_D14.16
- net ~{MBS}: no longer names the net of B_C12.10 (~{S})
- net ~{MBS}: now also B_F14.18
- net ~{OBJRAM}: no longer names the net of B_B13.6 (O2)
- net ~{OBJRAM}: now also B_B14.15
Other:
- note removed: "27"
- note removed: "29"
- note removed: "31"
- note removed: "33"
- note removed: "35"
- note removed: "38"
- note removed: "Add tri-state to verilog data signals and check delay on PCB"
- note removed: "BYT SYMBOL, till 501 jtkicad"
- note removed: "B_D14 is D_15 in original PCB. The position on PCB is D14."
- note removed: "kolla om det är inverterade A0 och A1 som används."
- moved on the sheet: B17A, B17C, B17F, B17G, B17H, B_A13, B_A14A, B_A14B, B_A14C, B_A14D, B_A14F, B_A14G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
