File: cores/mzone/sch/color_mixer.kicad_sch (KiCad schematic)
At the start: 18 parts

Commit message: mzone core
Connections:
- net PXLCLK renamed PXCK2'
Changed lines of the file:
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@@
 	(label "R1"
 		(at 274.32 149.86 0)
+		(fields_autoplaced yes)
 		(effects
 			(font
@@
 	(label "OCOL0"
 		(at 160.02 143.51 0)
+		(fields_autoplaced yes)
 		(effects
 			(font
@@
 	(label "R0"
 		(at 274.32 147.32 0)
+		(fields_autoplaced yes)
 		(effects
 			(font
@@
 	(label "G2"
 		(at 274.32 160.02 0)
+		(fields_autoplaced yes)
 		(effects
 			(font
@@
 	(label "B0"
 		(at 274.32 162.56 0)
+		(fields_autoplaced yes)
 		(effects
 			(font
@@
 	(label "TCOL''2"
 		(at 160.02 161.29 0)
+		(fields_autoplaced yes)
 		(effects
 			(font
@@
 	(label "G2"
 		(at 276.86 132.08 0)
+		(fields_autoplaced yes)
 		(effects
 			(font
@@
 	(label "R0"
 		(at 276.86 119.38 0)
+		(fields_autoplaced yes)
 		(effects
 			(font
@@
 	(label "B1"
 		(at 276.86 137.16 0)
+		(fields_autoplaced yes)
 		(effects
 			(font
@@
 	(label "TCOL''3"
 		(at 160.02 163.83 0)
+		(fields_autoplaced yes)
 		(effects
 			(font
@@
 	(label "G1"
 		(at 276.86 129.54 0)
+		(fields_autoplaced yes)
 		(effects
 			(font
@@
 	(label "G0"
 		(at 276.86 127 0)
+		(fields_autoplaced yes)
 		(effects
 			(font
@@
 	(label "R2"
 		(at 276.86 124.46 0)
+		(fields_autoplaced yes)
 		(effects
 			(font
@@
 	(label "TCOL''1"
 		(at 160.02 158.75 0)
+		(fields_autoplaced yes)
 		(effects
 			(font
@@
 	(label "R1"
 		(at 276.86 121.92 0)
+		(fields_autoplaced yes)
 		(effects
 			(font
@@
 	(label "B1"
 		(at 274.32 165.1 0)
+		(fields_autoplaced yes)
 		(effects
 			(font
@@
 	(label "TCOL''0"
 		(at 160.02 156.21 0)
-		(effects
-			(font
-				(size 1.27 1.27)
-			)
-			(justify left bottom)
-		)
-	)
-	(label "PXLCLK"
+		(fields_autoplaced yes)
+		(effects
+			(font
+				(size 1.27 1.27)
+			)
+			(justify left bottom)
+		)
+	)
+	(label "PXCK2'"
 		(at 203.2 165.1 0)
+		(fields_autoplaced yes)
 		(effects
 			(font
@@
 	(label "OCOL2"
 		(at 160.02 148.59 0)
+		(fields_autoplaced yes)
 		(effects
 			(font
@@
 	(label "B0"
 		(at 276.86 134.62 0)
+		(fields_autoplaced yes)
 		(effects
 			(font
@@
 	(label "R2"
 		(at 274.32 152.4 0)
+		(fields_autoplaced yes)
 		(effects
 			(font
@@
 	(label "OCOL1"
 		(at 160.02 146.05 0)
+		(fields_autoplaced yes)
 		(effects
 			(font
@@
 	(label "OCOL3"
 		(at 160.02 151.13 0)
+		(fields_autoplaced yes)
 		(effects
 			(font
@@
 	(label "G1"
 		(at 274.32 157.48 0)
+		(fields_autoplaced yes)
 		(effects
 			(font
@@
 	(label "G0"
 		(at 274.32 154.94 0)
+		(fields_autoplaced yes)
 		(effects
 			(font
@@
 		(shape input)
 		(at 154.94 140.97 180)
+		(fields_autoplaced yes)
 		(effects
 			(font
@@
 		(shape input)
 		(at 115.57 176.53 180)
+		(fields_autoplaced yes)
 		(effects
 			(font
@@
 		(shape output)
 		(at 300.99 167.64 0)
+		(fields_autoplaced yes)
 		(effects
 			(font
@@
 		(shape input)
 		(at 146.05 179.07 180)
+		(fields_autoplaced yes)
 		(effects
 			(font
@@
 		(shape input)
 		(at 146.05 170.18 180)
+		(fields_autoplaced yes)
 		(effects
 			(font
@@
 		(shape output)
 		(at 300.99 140.97 0)
+		(fields_autoplaced yes)
 		(effects
 			(font
@@
 		(shape input)
 		(at 146.05 165.1 180)
+		(fields_autoplaced yes)
 		(effects
 			(font
@@
 		(shape input)
 		(at 154.94 153.67 180)
+		(fields_autoplaced yes)
 		(effects
 			(font
@@
 		(shape output)
 		(at 300.99 154.94 0)
-		(effects
-			(font
+		(fields_autoplaced yes)
+		(effects
+			(font
