File: cores/mzone/sch/objects2.kicad_sch (KiCad schematic)
At the start: 16 parts

Commit message: mzone core
Connections:
- net CLK1 renamed PXCK1
- net CLK2 renamed PXCK2
- net M18DIV2 renamed OPCK
Other:
- note added: "PXCK2 is phase shifted 120deg in respect to PXCK1"
- note removed: "CLK2 is phase shifted 120deg in respect to CLK1"

Commit message: mzone core
Parts:
- removed A1: 74LS244, symbol jt74:74LS244
- added A1: 74LS244, symbol 74xx:74LS244_Split
Connections:
- net GND: now also A1.1, A1.10 (GND), A1.19
- net OCLK1: now also A1.11
- net OCLK2: now also A1.6
- net VCC: now also A1.20 (VCC)
- net ~{OBWR1}: no longer names the net of B4.10 (~{WR})
- net ~{OBWR1}: now also A1.9
- net ~{OBWR2}: no longer names the net of A4.10 (~{WR})
- net ~{OBWR2}: now also A1.14
- net ~{ODB}5L1 renamed ~{ODB5L}1
- net ~{ODB}5L2 renamed ~{ODB5L}2
- no-connect marks 12 -> 15
Other:
- note added: "Line buffers At the end of the read cycle, zeroes are written to RAM.?"
- note added: "Transp pixel: 4'b0000"
- note removed: "55ns hold time? check MBM2148L-55"
- note removed: "Kolla anslutningar från C2 till A1"
- note removed: "Kolla på PCB, anslutningar"
- note removed: "Line buffers At the end of the read cycle, zeroes are written to RAM."
- note removed: "OCLK1 and OCLK2 are pixel clocks."
- note removed: "White pixel: 4'b1111 Transparent pixel: 4'b0000"
- note removed: "http://www.bitsavers.org/components/fujitsu/_dataBooks/1982_Fujitsu_Memory_DatB_Book.pdf"
- note removed: "ok"
- note removed: "~{OSEL} is active if any of the ~{COL}XX are low -> ~{OSEL}1 or ~{OSEL}2 is active if the pixel is not transparetn. If the pixel is transparent the color value is taken from the LS735 for some reason."
- moved on the sheet: A4, A5, A6, A7, B1, B4, B5, B6, B7, C1A, C1D, C2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
