File: cores/mzone/sch/objects2.kicad_sch (KiCad schematic)
At the start: 16 parts

Commit message: mzone core
Parts:
- added unit 2 of A4
- added unit 2 of B4
- added unit 3 of C7
Connections:
- net GND: now also A4.9 (GND), B4.9 (GND), C7.7 (GND); no longer A4.9 (GND), B4.9 (GND)
- net VCC: now also A4.18 (VCC), B4.18 (VCC), C7.14 (VCC); no longer A4.18 (VCC), B4.18 (VCC)
Other:
- company: (none) -> Konami GX319
- title: (none) -> Megazone
