File: cores/mzone/sch/shram.kicad_sch (KiCad schematic)
At the start: 10 parts

Commit message: mzone core
Connections:
- net AB10 renamed MA'10
- net AB8 renamed MA'8
- net AB9 renamed MA'9
- net AS0 renamed SA0
- net AS1 renamed SA1
- net AS10 renamed SA10
- net AS2 renamed SA2
- net AS3 renamed SA3
- net AS4 renamed SA4
- net AS5 renamed SA5
- net AS6 renamed SA6
- net AS7 renamed SA7
- net AS8 renamed SA8
- net AS9 renamed SA9
- net BA0 renamed MA'0
- net BA1 renamed MA'1
- net BA2 renamed MA'2
- net BA3 renamed MA'3
- net BA4 renamed MA'4
- net BA5 renamed MA'5
- net BA6 renamed MA'6
- net BA7 renamed MA'7
- net ~{SVRAM} renamed ~{SSHRAM}
